File: Schematics.kicad_sch (KiCad schematic)
At the start: 70 parts, among them Q1 AO3400A, Q2 SI2301CDS-T1-E3, Q3 SI2301CDS-T1-E3, Q4 8050

Commit message: added raspberry pi footprint and README
Parts:
- added UP1: (no value), symbol Hat_Eink_Esp32:Eink_Esp32_Rpi
- C28: value 22nF/50V -> NC
Connections:
- net 3V3_OUT: now also C23.2, U3. (NC)
- net EPD_BUSY': now also UP1. (GPIO29)
- net EPD_CS': now also UP1. (GPIO29)
- net EPD_DC': now also UP1. (GPIO29)
- net EPD_DIN': now also UP1. (GPIO29)
- net EPD_RST': now also UP1. (GPIO29)
- net EPD_SCK': now also UP1. (GPIO29)
- net GND: now also UP1. (GPIO29)
- net PWR: now also 10K.1, NC/47K.1, UP1. (GPIO29)
- net SCL0: now also UP1. (GPIO29)
- net SDA0: now also UP1. (GPIO29)
- net VCC: now also Q3.3 (D)
- net VCC_INT: now also 47K.1, C22.2, NC/47K.2, Q3.2 (S)
- net VPC: now reaches C16.2, D4.2 (A)
- removed net +3.3V: C23.2, U3. (NC)
- new net RPI_3V3: UP1. (GPIO29)
- new net RPI_5V: UP1. (GPIO29)
- no-connect marks 0 -> 19

Commit message: added few footprints
Parts:
- removed C24: 100nF/50V, Capacitor_SMD:C_0603_1608Metric, symbol Device:C_Small
- removed U4: (no value), symbol Hat_Eink_Esp32:Eink_Esp32_TXB0108PWR
- added C33: 100nF/50V, Capacitor_SMD:C_0603_1608Metric, symbol Device:C_Small
- added U6: TXB0108PWR, local:TSSOP-20_L6.5-W4.4-P0.65-LS6.4-BL, symbol local:TXB0108PWR
- D1, D2, D3, D4: footprint (none) -> local:SOD-123_L2.8-W1.8-LS3.7-RD
- L3, L4: footprint (none) -> local:L0603
- Q1, Q4: footprint Package_TO_SOT_SMD:SOT-23 -> local:SOT-23-3_L2.9-W1.3-P1.90-LS2.4-BR
- Q2: footprint (none) -> local:SOT-23_L2.9-W1.3-P1.90-LS2.4-BR
- U3: footprint (none) -> local:SOT-23-5_L3.0-W1.7-P0.95-LS2.8-BR
- renumbered 0.2MΩ to 0.2M1, 0R to 0R1, 0R to 0R2, 0R to 0R3, 100K to 100K1, 10K to 10K1, 1K to 1K1, 1MΩ to 1M1, 3.9KΩ to 3.9K1, 3.9KΩ to 3.9K2, 47K to 47K1, C16 to C24, C23 to C27, NC/47K to NC/47K1, NC to NC1, NC to NC2, NC to NC3
Connections:
- net 3V3_OUT: now also C25.1, U6.10 (OE), U6.2 (VCCA); no longer C25.2
- net EPD_BUSY: now also U6.13 (B7)
- net EPD_BUSY': now also U6.8 (A7)
- net EPD_CS: now also U6.16 (B4)
- net EPD_CS': now also U6.5 (A4)
- net EPD_DC: now also U6.15 (B5)
- net EPD_DC': now also U6.6 (A5)
- net EPD_DIN: now also U6.18 (B2)
- net EPD_DIN': now also U6.3 (A2)
- net EPD_RST: now also U6.14 (B6)
- net EPD_RST': now also U6.7 (A6)
- net EPD_SCK: now also U6.17 (B3)
- net EPD_SCK': now also U6.4 (A3)
- net GND: now also C25.2, C33.2, U6.11 (GND); no longer C25.1
- net VCC: now also C33.1, U6.19 (VCCB)
Other:
- moved on the sheet: C25

Commit message: Assign footprints to all components and started pcb layout and connessions
Parts:
- removed U2: (no value), symbol Hat_Eink_Esp32:Eink_Esp32_Connector_9
- added P2: (no value), local:CONN-SMD_9P-P1.25_MOLEX_532610971, symbol Hat_Eink_Esp32:Eink_Esp32_Connector_9
- added R18, R19: NC, Resistor_SMD:R_0402_1005Metric, symbol Device:R_Small
- J1: footprint Connector_FFC-FPC:Amphenol_F32Q-1A7x1-11050_1x50-1MP_P0.5mm_Horizontal -> local:FPC-SMD_50P-P0.50_FPC0.5-WFB11-50P111-H20
- J2: footprint (none) -> Connector_PinSocket_2.54mm:PinSocket_1x03_P2.54mm_Vertical
- L1, L2: footprint (none) -> Inductor_SMD:L_1008_2520Metric
- Q3: footprint (none) -> local:SOT-23_L2.9-W1.3-P1.90-LS2.4-BR
- R1: renamed from 0R1; value R1 -> 0R
- R10: renamed from NC2; value R10 -> NC
- R11: renamed from 100K1; value R11 -> 100K
- R12: renamed from 1K1; value R12 -> 1K
- R13: renamed from 3.9K1; value R13 -> 3.9K
- R14: renamed from NC3; value R12 -> NC
- R15: renamed from 3.9K2; value R15 -> 3.9K
- R16: renamed from 0R2; value R16 -> 0R
- R17: renamed from 0R3; value R17 -> 0R
- R4: renamed from 1M1; value R4 -> 1MΩ
- R5: renamed from 0.2M1; value R5 -> 0.2Ω
- R6: renamed from 47K1; value R6 -> 47K
- R7: renamed from NC/47K1; value R7 -> NC/47K
- R8: renamed from 10K1; value R8 -> 10K
- R9: renamed from NC1; value R9 -> NC
- U5: value (none) -> CAT24C32; footprint (none) -> local:SOIC-8_L5.0-W4.0-P1.27-LS6.0-BL
- UP1: footprint (none) -> Connector_PinHeader_2.54mm:PinHeader_2x20_P2.54mm_Horizontal
- renumbered C24 to C16, C16 to C17, C17 to C18, C18 to C20, C25 to C24, C33 to C25
Connections:
- net 3V3_OUT: now also J2.1, U3.5 (VOUT), R18.1; no longer J2. (0), U3. (NC)
- net BS0: now also J2.2 (BS); no longer J2. (0)
- net EEPROM_VCC: now also U5.8 (VCC), R18.2, R19.2; no longer U5. (SDA)
- net EPD_BUSY: now also P2.8
- net EPD_BUSY': now also UP1.17 (GPIO5); no longer UP1. (GPIO29)
- net EPD_CS: now also P2.5
- net EPD_CS': now also UP1.23 (CE0); no longer UP1. (GPIO29)
- net EPD_DC: now also P2.6
- net EPD_DC': now also UP1.21 (GPIO6); no longer UP1. (GPIO29)
- net EPD_DIN: now also P2.3
- net EPD_DIN': now also UP1.20 (MOSI); no longer UP1. (GPIO29)
- net EPD_RST: now also P2.7
- net EPD_RST': now also UP1.12 (GPIO0); no longer UP1. (GPIO29)
- net EPD_SCK: now also P2.4
- net EPD_SCK': now also UP1.24 (SCLK); no longer UP1. (GPIO29)
- net GND: now also J2.3 (0), U3.2 (GND), U5.3 (A2), U5.4 (GND), UP1.10 (GND), UP1.13 (GND), UP1.19 (GND), UP1.26 (GND), UP1.29 (GND), UP1.33 (GND), UP1.40 (GND), UP1.5 (GND), P2.2; no longer J2. (0), U3. (NC), U5. (SDA), UP1. (GPIO29)
- net PWR: now also U3.3 (CE), UP1.11 (GPIO1), P2.9; no longer U3. (NC), UP1. (GPIO29)
- net RPI_3V3: now also UP1.18 (3V3), UP1.2 (3V3), R19.1; no longer UP1. (GPIO29)
- net RPI_5V: now also UP1.1 (5V), UP1.3 (5V); no longer UP1. (GPIO29)
- net SCL0: now also U5.6 (SCL), UP1.27 (SCL0); no longer U5. (SDA), UP1. (GPIO29)
- net SDA0: now also U5.5 (SDA), UP1.28 (SDA0); no longer U5. (SDA), UP1. (GPIO29)
- net VCC: now also U3.1 (VIN); no longer U3. (NC)
- net VCC_INT: now also P2.1
- net at R12.2, R14.1: now also U5.7 (WP); no longer U5. (SDA)
- net at R16.1, R9.2: now also U5.2 (A1); no longer U5. (SDA)
- net at C28.2: now also U3.4 (NC); no longer U3. (NC)
- net at R10.2, R17.1: now also U5.1 (A0); no longer U5. (SDA)

Commit message: completed PCB Layout
Parts:
- R1, R10, R11, R12, R13, R14, R15, R16, R17, R18, R19, R2, R20, R21, R22, R23, R3, R4, R5, R6, R7, R8, R9: footprint Resistor_SMD:R_0402_1005Metric -> Resistor_SMD:R_0603_1608Metric
- UP1: footprint Connector_PinHeader_2.54mm:PinHeader_2x20_P2.54mm_Horizontal -> local:HDR-SMD_40P-P2.54-V-F-R2-C20-S2.54-LS7.1
- renumbered U5 to U2
Connections:
- net 3.3V_OUT is gone; now on net EPD_3V3: C19.1, R21.2, R22.2
- net VCC_INT is gone; now on net RPI_5V: C22.2, P2.1, Q3.2 (S), R6.1, R7.2
- net 3V3_OUT: no longer J2.1
- net GDRC: now also J1.9 (GDRC); no longer J1.10 (RESEC)
- net RESEC: now also J1.10 (RESEC); no longer J1.11 (VPC)
- net VDD: now also J2.1
- net VPC: now also J1.11 (VPC)
Changed lines of the file:
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@@
 	(wire
 		(pts
+			(xy 44.45 48.26) (xy 50.8 48.26)
+		)
+		(stroke
+			(width 0)
+			(type default)
+		)
+	)
+	(wire
+		(pts
 			(xy 149.86 35.56) (xy 149.86 45.72)
 		)
@@
 	(wire
 		(pts
+			(xy 234.95 76.2) (xy 250.19 76.2)
+		)
+		(stroke
+			(width 0)
+			(type default)
+		)
+	)
+	(wire
+		(pts
 			(xy 49.53 124.46) (xy 49.53 157.48)
 		)
@@
 		)
 	)
+	(label "RPI_5V"
+		(at 250.19 76.2 0)
+		(effects
+			(font
+				(size 1.27 1.27)
+			)
+			(justify left bottom)
+		)
+	)
 	(label "VSH_LV2"
 		(at 50.8 68.58 0)
@@
 		)
 	)
-	(label "RESEC"
+	(label "VPC"
 		(at 50.8 53.34 0)
 		(effects
@@
 		)
 	)
+	(label "GDRC"
+		(at 50.8 48.26 0)
+		(effects
+			(font
+				(size 1.27 1.27)
+			)
+			(justify left bottom)
+		)
+	)
 	(label "VCP2"
 		(at 50.8 129.54 0)
@@
 		)
 	)
+	(label "VCC_INT"
+		(at 234.95 76.2 0)
+		(effects
+			(font
+				(size 1.27 1.27)
+			)
+			(justify left bottom)
+		)
+	)
 	(label "EPD_CS'"
 		(at 50.8 104.14 0)
@@
 		)
 	)
-	(label "GDRC"
+	(label "RESEC"
 		(at 50.8 50.8 0)
 		(effects
@@
 			)
 		)
-		(property "Footprint" "Resistor_SMD:R_0402_1005Metric"
+		(property "Footprint" "Resistor_SMD:R_0603_1608Metric"
 			(at 278.13 92.71 0)
 			(hide yes)
@@
 			)
 		)
-		(property "Footprint" "Resistor_SMD:R_0402_1005Metric"
+		(property "Footprint" "Resistor_SMD:R_0603_1608Metric"
 			(at 278.13 104.14 0)
 			(hide yes)
@@
 		)
 		(property "Value" "EEPROM_VCC"
-			(at 273.812 108.712 0)
+			(at 272.542 108.204 0)
 			(show_name no)
 			(do_not_autoplace no)
@@
 			)
 		)
-		(property "Footprint" "Resistor_SMD:R_0402_1005Metric"
+		(property "Footprint" "Resistor_SMD:R_0603_1608Metric"
 			(at 227.33 91.44 0)
 			(hide yes)
@@
 			)
 		)
-		(property "Footprint" "Resistor_SMD:R_0402_1005Metric"
+		(property "Footprint" "Resistor_SMD:R_0603_1608Metric"
 			(at 144.78 133.35 0)
 			(hide yes)
@@
 			)
 		)
-		(property "Footprint" "Resistor_SMD:R_0402_1005Metric"
+		(property "Footprint" "Resistor_SMD:R_0603_1608Metric"
 			(at 180.34 92.71 0)
 			(hide yes)
@@
 			)
 		)
-		(property "Footprint" "Resistor_SMD:R_0402_1005Metric"
+		(property "Footprint" "Resistor_SMD:R_0603_1608Metric"
 			(at 232.41 102.87 0)
 			(hide yes)
@@
 		)
 		(property "Value" "GND"
-			(at 238.76 110.744 0)
+			(at 239.268 110.998 0)
 			(show_name no)
 			(do_not_autoplace no)
@@
 			)
 		)
-		(property "Footprint" "Resistor_SMD:R_0402_1005Metric"
+		(property "Footprint" "Resistor_SMD:R_0603_1608Metric"
 			(at 60.96 152.4 0)
 			(hide yes)
@@
 			)
 		)
-		(property "Footprint" "Resistor_SMD:R_0402_1005Metric"
+		(property "Footprint" "Resistor_SMD:R_0603_1608Metric"
 			(at 57.15 33.02 0)
 			(hide yes)
@@
 			)
 		)
-		(property "Footprint" "Resistor_SMD:R_0402_1005Metric"
+		(property "Footprint" "Resistor_SMD:R_0603_1608Metric"
 			(at 144.78 139.7 0)
 			(hide yes)
@@
 		)
 		(property "Value" "EEPROM_VCC"
-			(at 239.268 86.36 90)
+			(at 239.522 84.074 90)
 			(show_name no)
 			(do_not_autoplace no)
@@
 			)
 		)
-		(property "Footprint" "Resistor_SMD:R_0402_1005Metric"
+		(property "Footprint" "Resistor_SMD:R_0603_1608Metric"
 			(at 265.43 101.6 0)
 			(hide yes)
@@
 			)
 		)
-		(property "Footprint" "Resistor_SMD:R_0402_1005Metric"
+		(property "Footprint" "Resistor_SMD:R_0603_1608Metric"
 			(at 104.14 44.45 0)
 			(hide yes)
@@
 			)
 		)
-		(property "Footprint" "Resistor_SMD:R_0402_1005Metric"
+		(property "Footprint" "Resistor_SMD:R_0603_1608Metric"
 			(at 114.3 44.45 0)
 			(hide yes)
@@
 		)
 		(property "Value" "GND"
-			(at 229.87 110.744 0)
+			(at 230.632 110.998 0)
 			(show_name no)
 			(do_not_autoplace no)
@@
 			)
 		)
-		(property "Footprint" "Resistor_SMD:R_0402_1005Metric"
+		(property "Footprint" "Resistor_SMD:R_0603_1608Metric"
 			(at 232.41 91.44 0)
 			(hide yes)
@@
 			)
 		)
-		(property "Value" "3.3V_OUT"
+		(property "Value" "EPD_3V3"
 			(at 79.502 118.11 0)
 			(show_name no)
@@
 			)
 		)
-		(property "Footprint" "Resistor_SMD:R_0402_1005Metric"
+		(property "Footprint" "Resistor_SMD:R_0603_1608Metric"
 			(at 179.07 107.95 0)
 			(hide yes)
@@
 		)
 		(property "Value" "VCC"
-			(at 202.438 85.09 90)
+			(at 199.898 83.312 90)
 			(show_name no)
 			(do_not_autoplace no)
@@
 			)
 		)
-		(property "Footprint" "Resistor_SMD:R_0402_1005Metric"
+		(property "Footprint" "Resistor_SMD:R_0603_1608Metric"
 			(at 115.57 102.87 0)
 			(hide yes)
@@
 			)
 		)
-		(property "Footprint" "Resistor_SMD:R_0402_1005Metric"
+		(property "Footprint" "Resistor_SMD:R_0603_1608Metric"
 			(at 168.91 105.41 0)
 			(hide yes)
@@
 			)
 		)
-		(property "Footprint" "Resistor_SMD:R_0402_1005Metric"
+		(property "Footprint" "Resistor_SMD:R_0603_1608Metric"
 			(at 227.33 102.87 0)
 			(hide yes)
@@
 			)
 		)
-		(property "Footprint" "Resistor_SMD:R_0402_1005Metric"
+		(property "Footprint" "Resistor_SMD:R_0603_1608Metric"
 			(at 60.96 121.92 0)
 			(hide yes)
@@
 			)
 		)
-		(property "Footprint" "Connector_PinHeader_2.54mm:PinHeader_2x20_P2.54mm_Horizontal"
+		(property "Footprint" "local:HDR-SMD_40P-P2.54-V-F-R2-C20-S2.54-LS7.1"
 			(at 205.74 46.99 0)
 			(hide yes)
@@
 			)
 		)
-		(property "Footprint" "Resistor_SMD:R_0402_1005Metric"
+		(property "Footprint" "Resistor_SMD:R_0603_1608Metric"
 			(at 163.83 96.52 0)
 			(hide yes)
@@
 			)
 		)
-		(property "Footprint" "Resistor_SMD:R_0402_1005Metric"
+		(property "Footprint" "Resistor_SMD:R_0603_1608Metric"
 			(at 60.96 127 0)
 			(hide yes)
@@
 		(in_pos_files yes)
 		(dnp no)
-		(property "Reference" "U5"
+		(property "Reference" "U2"
 			(at 250.698 93.726 0)
 			(show_name no)
@@
 			(project "Schematics"
 				(path "/ba81e668-39a3-44b1-9436-fbe95b38ede8"
-					(reference "U5")
+					(reference "U2")
 					(unit 1)
 				)
@@
 			)
 		)
-		(property "Footprint" "Resistor_SMD:R_0402_1005Metric"
+		(property "Footprint" "Resistor_SMD:R_0603_1608Metric"
 			(at 158.75 25.4 0)
 			(hide yes)
@@
 			)
 		)
-		(property "Footprint" "Resistor_SMD:R_0402_1005Metric"
+		(property "Footprint" "Resistor_SMD:R_0603_1608Metric"
 			(at 97.79 80.01 0)
 			(hide yes)
@@
 		)
 		(property "Value" "EEPROM_VCC"
-			(at 273.304 82.55 0)
+			(at 272.288 82.55 0)
 			(show_name no)
 			(do_not_autoplace no)
@@
 			)
 		)
-		(property "Footprint" "Resistor_SMD:R_0402_1005Metric"
+		(property "Footprint" "Resistor_SMD:R_0603_1608Metric"
 			(at 265.43 104.14 0)
 			(hide yes)
@@
 		)
 		(property "Value" "SI2301CDS-T1-E3"
-			(at 191.77 88.9 90)
+			(at 192.278 88.9 90)
 			(show_name no)
 			(do_not_autoplace no)
@@
 			)
 		)
-		(property "Value" "3V3_OUT"
+		(property "Value" "VDD"
 			(at 200.152 62.992 90)
 			(show_name no)

Commit message: fixed minor connection mistakes/errors, and added BOM and POS files
Parts:
- C2, C21: value 470uF/25V -> 470nF/25V
- C24, C25, C27: value 100nF/50V -> 1uF/50V
- C29: footprint Capacitor_SMD:C_0603_1608Metric -> Capacitor_SMD:C_1206_3216Metric
- Q4: footprint local:SOT-23-3_L2.9-W1.3-P1.90-LS2.4-BR -> local:SOT-23-3_L3.0-W1.7-P0.95-LS2.9-BR
- R13, R15: value 3.9K -> 3.9KΩ
- R19: value NC -> 0R
- R3: value 0.2MΩ -> 0.2Ω
- U3: value (none) -> ME6217C33M5G
Changed lines of the file:
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@@
 		(in_pos_files yes)
 		(dnp no)
-		(fields_autoplaced yes)
 		(property "Reference" "P2"
-			(at 27.94 168.91 0)
-			(hide yes)
+			(at 28.956 164.592 0)
 			(show_name no)
 			(do_not_autoplace no)
@@
 		(in_pos_files yes)
 		(dnp no)
-		(fields_autoplaced yes)
 		(property "Reference" "U3"
-			(at 116.205 166.37 0)
+			(at 115.824 167.386 0)
 			(show_name no)
 			(do_not_autoplace no)
@@
 			)
 		)
-		(property "Value" ""
-			(at 107.95 171.45 0)
+		(property "Value" "ME6217C33M5G"
+			(at 116.332 178.054 0)
 			(show_name no)
 			(do_not_autoplace no)
@@
 			)
 		)
-		(property "Value" "100nF/50V"
+		(property "Value" "1uF/50V"
 			(at 141.224 164.846 0)
 			(show_name no)
@@
 			)
 		)
-		(property "Footprint" "local:SOT-23-3_L2.9-W1.3-P1.90-LS2.4-BR"
+		(property "Footprint" "local:SOT-23-3_L3.0-W1.7-P0.95-LS2.9-BR"
 			(at 191.77 112.776 0)
 			(hide yes)
@@
 			)
 		)
-		(property "Value" "NC"
+		(property "Value" "0R"
 			(at 143.764 141.478 90)
 			(show_name no)
@@
 			)
 		)
-		(property "Value" "3.9K"
+		(property "Value" "3.9KΩ"
 			(at 270.256 100.584 90)
 			(show_name no)
@@
 			)
 		)
-		(property "Value" "0.2MΩ"
+		(property "Value" "0.2Ω"
 			(at 117.856 45.72 0)
 			(show_name no)
@@
 			)
 		)
-		(property "Value" "470uF/25V"
+		(property "Value" "470nF/25V"
 			(at 69.8563 29.21 90)
 			(show_name no)
@@
 			)
 		)
-		(property "Value" "100nF/50V"
+		(property "Value" "1uF/50V"
 			(at 195.58 136.398 0)
 			(show_name no)
@@
 		(dnp no)
 		(property "Reference" "U6"
-			(at 231.14 121.92 0)
+			(at 232.41 120.65 0)
 			(show_name no)
 			(do_not_autoplace no)
@@
 		)
 		(property "Value" "TXB0108PWR"
-			(at 231.14 124.46 0)
+			(at 233.172 123.952 0)
 			(show_name no)
 			(do_not_autoplace no)
@@
 		(dnp no)
 		(property "Reference" "R1"
-			(at 158.75 27.178 90)
+			(at 159.004 23.876 90)
 			(show_name no)
 			(do_not_autoplace no)
@@
 		)
 		(property "Value" "0R"
-			(at 158.75 23.622 90)
+			(at 158.75 27.178 90)
 			(show_name no)
 			(do_not_autoplace no)
@@
 			)
 		)
-		(property "Value" "100nF/50V"
-			(at 268.478 135.636 0)
+		(property "Value" "1uF/50V"
+			(at 265.43 135.382 0)
 			(show_name no)
 			(do_not_autoplace no)
@@
 			)
 		)
-		(property "Value" "470uF/25V"
+		(property "Value" "470nF/25V"
 			(at 68.58 154.94 90)
 			(show_name no)
@@
 			)
 		)
-		(property "Value" "3.9K"
+		(property "Value" "3.9KΩ"
 			(at 269.748 103.378 90)
 			(show_name no)
@@
 			)
 		)
-		(property "Footprint" "Capacitor_SMD:C_0603_1608Metric"
+		(property "Footprint" "Capacitor_SMD:C_1206_3216Metric"
 			(at 193.04 35.56 0)
 			(hide yes)
